Commit message: updated gazebo modules

File: src/kuka_iiwa/kuka_iiwa_description/urdf/iiwa_gripper.urdf (robot description, URDF)
Before this commit: robot iiwa14_gripper::iiwa14, 13 links, 12 joints
Links:
- added link left_cube, mass 1e-5
- added link right_cube, mass 1e-5
Joints:
- added joint left_end: type revolute, parent gripper_left_link, child left_cube, origin xyz=0 0 -0.160 rpy=0 0 0, axis 0 0 0, limit lower=0.0000010 upper=0.0000011 effort=0 velocity=0
- added joint right_end: type revolute, parent gripper_right_link, child right_cube, origin xyz=0 0 -0.160 rpy=0 0 0, axis 0 0 0, limit lower=0.0000010 upper=0.0000011 effort=0 velocity=0
